Commit message: VREP Simulation is working

File: src/ackermann_vehicle-1/ackermann_vehicle_description/urdf/em_3905.urdf.xacro (robot description, xacro)
@@ -29,25 +29,24 @@
 <robot name="em_3905" xmlns:xacro="http://www.ros.org/wiki/xacro">
   <!-- Degree-to-radian conversions -->
-  <xacro:property name="degrees_45" value=".42195"/> <!-- Changed from 0.785398163, for max turn radius using this paper, pages 25 - 27, "Automatic_Steering_Methods_for_Autonomous_Automobile_Path_Tracking.pdf", Tyler Proffitt -->
+  <xacro:property name="degrees_45" value="0.785398163"/>
   <xacro:property name="degrees_90" value="1.57079633"/>
   <!-- chassis_length is measured along the x axis, chassis_width
        along the y axis, and chassis_height along the z axis. -->
-  <xacro:property name="chassis_length" value="2.97"/>   <!-- Changed from 0.258, Tyler Proffitt -->
-  <xacro:property name="chassis_width" value="1.54"/>    <!-- Changed from 0.168, Tyler Proffitt -->
+  <xacro:property name="chassis_length" value="0.258"/>
+  <xacro:property name="chassis_width" value="0.168"/>
   <xacro:property name="chassis_height" value="0.01"/>
-  <xacro:property name="chassis_mass" value=".001"/>     <!-- Changed from 2.76, due to weird jumping on startup, Tyler Proffitt -->
+  <xacro:property name="chassis_mass" value="2.788"/>
   <!-- battery_dist is the distance between the inner edges of the
        batteries. battery_comp_depth is the battery compartment depth.
        battery_length is measured along the x axis, battery_width
        along the y axis, and battery_height along the z axis. -->
-  <!-- Changed to zero out, Tyler Proffitt -->
-  <xacro:property name="battery_x_offset" value="0"/>
-  <xacro:property name="battery_dist" value="0"/>
-  <xacro:property name="battery_comp_depth" value="-.25"/>
-  <xacro:property name="battery_comp_angle" value="0"/>
-  <xacro:property name="battery_length" value=".25"/>
-  <xacro:property name="battery_width" value=".25"/>
-  <xacro:property name="battery_height" value=".25"/>
-  <xacro:property name="battery_mass" value="0.001"/>
+  <xacro:property name="battery_x_offset" value="0.055"/>
+  <xacro:property name="battery_dist" value="0.065"/>
+  <xacro:property name="battery_comp_depth" value="0.02"/>
+  <xacro:property name="battery_comp_angle" value="0.34906585"/>
+  <xacro:property name="battery_length" value="0.16"/>
+  <xacro:property name="battery_width" value="0.047"/>
+  <xacro:property name="battery_height" value="0.024"/>
+  <xacro:property name="battery_mass" value="0.5025"/>
   <!-- hub_dia and tire_dia are the diameters of the hub and tire,
        respectively. hex_hub_depth is the distance that the hex hub is
@@ -55,6 +54,6 @@
        is a "zero offset" wheel. hex_hub_depth = tire_width / 2 -
        axle_length. -->
-  <xacro:property name="hub_dia" value="0.3302"/>        <!-- Changed from 0.09652, Tyler Proffitt -->
-  <xacro:property name="tire_dia" value=".6604"/>        <!-- Changed from 0.14605, Tyler Proffitt -->
+  <xacro:property name="hub_dia" value="0.09652"/>
+  <xacro:property name="tire_dia" value="0.14605"/>
   <xacro:property name="tire_width" value="0.0889"/>
   <xacro:property name="hex_hub_depth" value="0.01445"/>
@@ -64,15 +63,15 @@
        from a U joint to the corresponding hex hub. wheel_travel is the
        vertical wheel travel. -->
-  <xacro:property name="wheelbase" value="2.065"/>       <!-- Changed from 0.335, Tyler Proffitt -->
-  <xacro:property name="hex_hub_dist" value="1.143"/>    <!-- Changed from 0.365, Tyler Proffitt -->
+  <xacro:property name="wheelbase" value="0.335"/>
+  <xacro:property name="hex_hub_dist" value="0.365"/>
   <xacro:property name="axle_length" value="0.03"/>
-  <xacro:property name="wheel_travel" value="0"/>        <!-- Changed, due to weird vibration during movement, Tyler Proffitt -->
-  <xacro:property name="shock_z_offset" value="0"/>      <!-- Changed, due to weird vibration during movement, Tyler Proffitt -->
+  <xacro:property name="wheel_travel" value="0.084"/>
+  <xacro:property name="shock_z_offset" value="0.0655"/>
   <!-- shock_eff_limit is 2 * ((shock_stroke / 2) * shock_spring_constant) N.
        shock_stroke is 0.028575 meters. shock_spring_constant, an approximation
        of a Traxxas Ultra Shock shock absorber spring's constant, is
        437.817 N/m. -->
-  <xacro:property name="shock_eff_limit" value=".0001"/> <!-- Changed from 12.5106, due to weird vibration on startup, Tyler Proffitt -->
-  <xacro:property name="shock_vel_limit" value=".0001"/> <!-- Changed from 1000, due to weird vibration on startup, Tyler Proffitt -->
+  <xacro:property name="shock_eff_limit" value="12.5106"/>
+  <xacro:property name="shock_vel_limit" value="1000"/>
   <!-- The specifications for a Titan(R) 550 motor could not be found, so the
        stall torque of a Mabuchi Motor(R) RS-550VC-7525 motor was used instead.
@@ -98,5 +97,5 @@
   </material>
   <material name="chassis_mat">
-    <color rgba="0 0 1 1"/>
+    <color rgba="0.5 0.5 0.5 1"/>
   </material>
   <material name="tire_mat">
@@ -342,5 +341,5 @@
   <link name="chassis">
     <visual>
-      <origin xyz="0 0 .29"/> <!-- Changed z comp. from ${-chassis_height / 2}, Tyler Proffitt -->
+      <origin xyz="0 0 ${-chassis_height / 2}"/>
       <geometry>
         <box size="${chassis_length} ${chassis_width} ${chassis_height}"/>
@@ -349,5 +348,5 @@
     </visual>
     <collision>
-      <origin xyz="0 0 .29"/> <!-- Changed z comp. from ${-chassis_height / 2}, Tyler Proffitt -->
+      <origin xyz="0 0 ${-chassis_height / 2}"/>
       <geometry>
         <box size="${chassis_length} ${chassis_width} ${chassis_height}"/>
@@ -357,5 +356,5 @@
         width="${chassis_length}" depth="${chassis_width}"
         height="${chassis_height}" mass="${chassis_mass}">
-      <origin xyz="0 0 .29"/> <!-- Changed z comp. from ${-chassis_height / 2}, Tyler Proffitt -->
+      <origin xyz="0 0 ${-chassis_height / 2}"/>
     </xacro:solid_cuboid_inertial>
   </link>
